Commit message: Update diffrobot.xacro

File: uvc_robot/urdf/diffrobot.xacro (robot description, xacro)
@@ -205,14 +205,14 @@
   <parent link="base_link"/>
     <child link="lidar_link"/>
-    <axis xyz="0.0 1.0 0.0"/>
-    <limit lower="0.0" upper="0.0" effort="0.0" velocity="0.0"/>
-</joint>
-    <!-- <link name="laser_data_link">
+    <axis xyz="0.0 0.0 0.0"/>
+    <limit lower="0.0" upper="0.0" effort="0.0" velocity="0.0"/>
+</joint>
+    <link name="laser_data_link">
     </link>
     <joint name="laser_data_joint" type="fixed">
-        <origin xyz="0.45 0.0 0.55" rpy="-1.5708 -0.0 -1.5708"/>
+        <origin xyz="0.0 0.0 0.0" rpy="0.0 -1.5708 -1.5708"/>
         <parent link="lidar_link"/>
         <child link="laser_data_link"/>
-    </joint> -->
+    </joint>
   <!-- Camera -->
   <link name="camera_link">
